Commit message: use the collision mesh to replace the visual mesh

File: tests/data/ur5/ur5.urdf (robot description, URDF)
Before this commit: robot ur5, 11 links, 10 joints
Links:
- link base_link: geometry collision mesh filename=collision/base.stl; visual mesh filename=collision/base.stl
- link forearm_link: geometry collision mesh filename=collision/forearm.stl; visual mesh filename=collision/forearm.stl
- link shoulder_link: geometry collision mesh filename=collision/shoulder.stl; visual mesh filename=collision/shoulder.stl
- link upper_arm_link: geometry collision mesh filename=collision/upperarm.stl; visual mesh filename=collision/upperarm.stl
- link wrist_1_link: geometry collision mesh filename=collision/wrist1.stl; visual mesh filename=collision/wrist1.stl
- link wrist_2_link: geometry collision mesh filename=collision/wrist2.stl; visual mesh filename=collision/wrist2.stl
- link wrist_3_link: geometry collision mesh filename=collision/wrist3.stl; visual mesh filename=collision/wrist3.stl
